Commit message: Finish Design

File: description/robot.urdf.xacro (robot description, xacro)
@@ -2,3 +2,4 @@
 <robot xmlns:xacro="http://www.ros.org/wiki/xacro"  name="robot">
     <xacro:include filename='robot_core.xacro'/>
+    <xacro:include filename='gazebo_control.xacro'/>
 </robot>

File: description/robot_core.xacro (robot description, xacro)
@@ -1,4 +1,5 @@
 <?xml version="1.0"?>
 <robot xmlns:xacro="http://www.ros.org/wiki/xacro" >
+    <xacro:include filename='inertial_macros.xacro'/>
     <!-- Materials determine-->
     <material name='white'>
@@ -38,4 +39,10 @@
         </collision>
     </link>
+    <xacro:inertial_box mass='0.5' x='1' y='0.7' z='0.5'>
+        <origin xyz= '0 0 0' rpy='0 0 0'/>
+    </xacro:inertial_box>
+    <gazebo reference='chassis'>
+        <material>Gazebo/white</material>
+    </gazebo>
     <!-- Wheels -->
     <!-- LEFT FRONT -->
@@ -59,4 +66,10 @@
         </collision>
     </link>
+    <xacro:inertial_cylinder mass='0.1' length='0.04' radius='0.15'>
+        <origin xyz= '0 0 0' rpy='0 0 0'/>
+    </xacro:inertial_cylinder>
+    <gazebo reference='left_front_wheel'>
+        <material>Gazebo/blue</material>
+    </gazebo>
     <!-- RIGHT FRONT -->
     <joint name="right_front_wheel_joint" type='continuous'>
@@ -79,4 +92,10 @@
         </collision>
     </link>
+    <xacro:inertial_cylinder mass='0.1' length='0.04' radius='0.15'>
+        <origin xyz= '0 0 0' rpy='0 0 0'/>
+    </xacro:inertial_cylinder>
+    <gazebo reference='right_front_wheel'>
+        <material>Gazebo/blue</material>
+    </gazebo>
     <!-- RIGHT REAR -->
     <joint name="right_rear_wheel_joint" type='continuous'>
@@ -99,4 +118,10 @@
         </collision>
     </link>
+    <xacro:inertial_cylinder mass='0.1' length='0.04' radius='0.15'>
+        <origin xyz= '0 0 0' rpy='0 0 0'/>
+    </xacro:inertial_cylinder>
+    <gazebo reference='right_rear_wheel'>
+        <material>Gazebo/blue</material>
+    </gazebo>
     <!-- LEFT REAR -->
     <joint name="left_rear_wheel_joint" type='continuous'>
@@ -119,3 +144,9 @@
         </collision>
     </link>
+    <xacro:inertial_cylinder mass='0.1' length='0.04' radius='0.15'>
+        <origin xyz= '0 0 0' rpy='0 0 0'/>
+    </xacro:inertial_cylinder>
+    <gazebo reference='left_rear_wheel'>
+        <material>Gazebo/blue</material>
+    </gazebo>
 </robot>

Commit message: Lidar + Update on files

File: description/robot.urdf.xacro (robot description, xacro)
@@ -3,3 +3,4 @@
     <xacro:include filename='robot_core.xacro'/>
     <xacro:include filename='gazebo_control.xacro'/>
+    <xacro:include filename='lidar.xacro'/>
 </robot>

File: description/robot_core.xacro (robot description, xacro)
@@ -65,8 +65,8 @@
             </geometry>
         </collision>
+        <xacro:inertial_cylinder mass='0.1' length='0.04' radius='0.15'>
+            <origin xyz= '0 0 0' rpy='0 0 0'/>
+        </xacro:inertial_cylinder>
     </link>
-    <xacro:inertial_cylinder mass='0.1' length='0.04' radius='0.15'>
-        <origin xyz= '0 0 0' rpy='0 0 0'/>
-    </xacro:inertial_cylinder>
     <gazebo reference='left_front_wheel'>
         <material>Gazebo/blue</material>
@@ -91,8 +91,8 @@
             </geometry>
         </collision>
+        <xacro:inertial_cylinder mass='0.1' length='0.04' radius='0.15'>
+            <origin xyz= '0 0 0' rpy='0 0 0'/>
+        </xacro:inertial_cylinder>
     </link>
-    <xacro:inertial_cylinder mass='0.1' length='0.04' radius='0.15'>
-        <origin xyz= '0 0 0' rpy='0 0 0'/>
-    </xacro:inertial_cylinder>
     <gazebo reference='right_front_wheel'>
         <material>Gazebo/blue</material>
@@ -117,8 +117,8 @@
             </geometry>
         </collision>
+        <xacro:inertial_cylinder mass='0.1' length='0.04' radius='0.15'>
+            <origin xyz= '0 0 0' rpy='0 0 0'/>
+        </xacro:inertial_cylinder>
     </link>
-    <xacro:inertial_cylinder mass='0.1' length='0.04' radius='0.15'>
-        <origin xyz= '0 0 0' rpy='0 0 0'/>
-    </xacro:inertial_cylinder>
     <gazebo reference='right_rear_wheel'>
         <material>Gazebo/blue</material>
@@ -143,8 +143,8 @@
             </geometry>
         </collision>
+        <xacro:inertial_cylinder mass='0.1' length='0.04' radius='0.15'>
+            <origin xyz= '0 0 0' rpy='0 0 0'/>
+        </xacro:inertial_cylinder>
     </link>
-    <xacro:inertial_cylinder mass='0.1' length='0.04' radius='0.15'>
-        <origin xyz= '0 0 0' rpy='0 0 0'/>
-    </xacro:inertial_cylinder>
     <gazebo reference='left_rear_wheel'>
         <material>Gazebo/blue</material>
