Commit message: lidar file fix

File: description/lidar.xacro (robot description, xacro)
@@ -4,10 +4,10 @@
         <parent link='chassis'/>
         <child link='lidar'/>
-        <origin xyz= '0.1 0 0.175' rpy= '0 0 0'/>
+        <origin xyz= '0.1 0 0.525' rpy= '0 0 0'/>
     </joint>
     <link name='lidar'>
         <visual>
             <geometry>
-                <cylinder radius='0.15' length='0.04'/>
+                <cylinder radius='0.05' length='0.04'/>
             </geometry>
             <material name='red'/>
@@ -15,5 +15,5 @@
         <collision>
             <geometry>
-                <cylinder radius='0.15' length='0.04'/>
+                <cylinder radius='0.05' length='0.04'/>
             </geometry>
         </collision>
