Commit message: 11/12 3

File: description/robot_core.xacro (robot description, xacro)
@@ -22,5 +22,5 @@
         <parent link='base_link'/>
         <child link='chassis'/>
-        <origin xyz=' 0 0 0'/>
+        <origin xyz='0 0 0'/>
     </joint>
     <link name='chassis'>
@@ -38,8 +38,8 @@
             </geometry>
         </collision>
+        <xacro:inertial_box mass='1.4' x='1' y='0.7' z='0.5'>
+            <origin xyz= '0 0 0' rpy='0 0 0'/>
+        </xacro:inertial_box>
     </link>
-    <xacro:inertial_box mass='1.4' x='1' y='0.7' z='0.5'>
-        <origin xyz= '0 0 0' rpy='0 0 0'/>
-    </xacro:inertial_box>
     <gazebo reference='chassis'>
         <material>Gazebo/White</material>
