Commit message: hard changes

File: description/gazebo_control.xacro (robot description, xacro)
@@ -1,14 +1,12 @@
 <?xml version="1.0"?>
-<robot xmlns:xacro="http://www.ros.org/wiki/xacro" >
+<robot xmlns:xacro="http://www.ros.org/wiki/xacro">
     <gazebo>
-        <plugin name='diff_drive' filename='libgazebo_ros_diffdrive.so'>
-            <!-- Wheel information -->
-            <left_front_joint>left_front_wheel_joint</left_front_joint>
-            <left_rear_joint>left_rear_wheel_joint</left_rear_joint>
-            <right_front_joint>right_front_wheel_joint</right_front_joint>
-            <right_rear_joint>right_rear_wheel_joint</right_rear_joint>
-            <wheel_separation>0.7</wheel_separation>
-            <wheel_diameter>0.15</wheel_diameter>
-            <!--Limits-->
+        <plugin name="diff_drive" filename="libgazebo_ros_diff_drive.so">
+            <!-- Wheel Information -->
+            <left_joint>left_wheel_joint</left_joint>
+            <right_joint>right_wheel_joint</right_joint>
+            <wheel_separation>0.297</wheel_separation>
+            <wheel_diameter>0.066</wheel_diameter>
+            <!-- Limits -->
             <max_wheel_torque>200</max_wheel_torque>
             <max_wheel_acceleration>10.0</max_wheel_acceleration>

File: description/lidar.xacro (robot description, xacro)
@@ -4,5 +4,5 @@
         <parent link='chassis'/>
         <child link='lidar'/>
-        <origin xyz= '0.1 0 0.175' rpy= '0 0 0'>
+        <origin xyz= '0.1 0 0.175' rpy= '0 0 0'/>
     </joint>
     <link name='lidar'>

File: description/robot_core.xacro (robot description, xacro)
@@ -65,5 +65,5 @@
             </geometry>
         </collision>
-        <xacro:inertial_cylinder mass='0.1' length='0.04' radius='0.15'>
+        <xacro:inertial_cylinder mass='0.01' length='0.04' radius='0.15'>
             <origin xyz= '0 0 0' rpy='0 0 0'/>
         </xacro:inertial_cylinder>
@@ -91,5 +91,5 @@
             </geometry>
         </collision>
-        <xacro:inertial_cylinder mass='0.1' length='0.04' radius='0.15'>
+        <xacro:inertial_cylinder mass='0.01' length='0.04' radius='0.15'>
             <origin xyz= '0 0 0' rpy='0 0 0'/>
         </xacro:inertial_cylinder>
@@ -117,5 +117,5 @@
             </geometry>
         </collision>
-        <xacro:inertial_cylinder mass='0.1' length='0.04' radius='0.15'>
+        <xacro:inertial_cylinder mass='0.01' length='0.04' radius='0.15'>
             <origin xyz= '0 0 0' rpy='0 0 0'/>
         </xacro:inertial_cylinder>
@@ -143,5 +143,5 @@
             </geometry>
         </collision>
-        <xacro:inertial_cylinder mass='0.1' length='0.04' radius='0.15'>
+        <xacro:inertial_cylinder mass='0.01' length='0.04' radius='0.15'>
             <origin xyz= '0 0 0' rpy='0 0 0'/>
         </xacro:inertial_cylinder>

Commit message: files fix

File: description/gazebo_control.xacro (robot description, xacro)
@@ -2,8 +2,10 @@
 <robot xmlns:xacro="http://www.ros.org/wiki/xacro">
     <gazebo>
-        <plugin name="diff_drive" filename="libgazebo_ros_diff_drive.so">
+        <plugin name="diff_drive" filename="libgazebo_ros_diff_ drive.so">
             <!-- Wheel Information -->
-            <left_joint>left_wheel_joint</left_joint>
-            <right_joint>right_wheel_joint</right_joint>
+            <left_front_wheel_joint>left_front_wheel_joint</left_front_wheel_joint>
+            <right_front_wheel_joint>right_front_wheel_joint</right_front_wheel_joint>
+            <left_rear_wheel_joint>left_rear_wheel_joint</left_rear_wheel_joint>
+            <right_rear_wheel_joint>right_rear_wheel_joint</right_rear_wheel_joint>
             <wheel_separation>0.297</wheel_separation>
             <wheel_diameter>0.066</wheel_diameter>

File: description/robot_core.xacro (robot description, xacro)
@@ -43,5 +43,5 @@
     </xacro:inertial_box>
     <gazebo reference='chassis'>
-        <material>Gazebo/white</material>
+        <material>Gazebo/White</material>
     </gazebo>
     <!-- Wheels -->
@@ -70,5 +70,7 @@
     </link>
     <gazebo reference='left_front_wheel'>
-        <material>Gazebo/blue</material>
+        <material>Gazebo/Blue</material>
+        <mu1 value="0.001"/>
+        <mu2 value="0.001"/>
     </gazebo>
     <!-- RIGHT FRONT -->
@@ -96,5 +98,7 @@
     </link>
     <gazebo reference='right_front_wheel'>
-        <material>Gazebo/blue</material>
+        <material>Gazebo/Blue</material>
+        <mu1 value="0.001"/>
+        <mu2 value="0.001"/>
     </gazebo>
     <!-- RIGHT REAR -->
@@ -122,5 +126,5 @@
     </link>
     <gazebo reference='right_rear_wheel'>
-        <material>Gazebo/blue</material>
+        <material>Gazebo/Blue</material>
     </gazebo>
     <!-- LEFT REAR -->
@@ -148,5 +152,5 @@
     </link>
     <gazebo reference='left_rear_wheel'>
-        <material>Gazebo/blue</material>
+        <material>Gazebo/Blue</material>
     </gazebo>
 </robot>

Commit message: hard 2811

File: description/gazebo_control.xacro (robot description, xacro)
@@ -2,5 +2,5 @@
 <robot xmlns:xacro="http://www.ros.org/wiki/xacro">
     <gazebo>
-        <plugin name="diff_drive" filename="libgazebo_ros_diff_ drive.so">
+        <plugin name="diff_drive" filename="libgazebo_ros_diff_drive.so">
             <!-- Wheel Information -->
             <left_front_wheel_joint>left_front_wheel_joint</left_front_wheel_joint>

File: description/lidar.xacro (robot description, xacro)
@@ -4,5 +4,5 @@
         <parent link='chassis'/>
         <child link='lidar'/>
-        <origin xyz= '0.1 0 0.525' rpy= '0 0 0'/>
+        <origin xyz= '0.1 0 0.275' rpy= '0 0 0'/>
     </joint>
     <link name='lidar'>
@@ -33,5 +33,5 @@
                         <samples>360</samples>
                         <resolution>1</resolution>
-                        <min_angle>3.14</min_angle>
+                        <min_angle>-3.14</min_angle>
                         <max_angle>3.14</max_angle>
                     </horizontal>
@@ -43,5 +43,5 @@
                 </range>
             </ray>
-            <plugin name='Lidar_controller' filename="libgazebo_ros_ray_sensor.so">
+            <plugin name='lidar_controller' filename="libgazebo_ros_ray_sensor.so">
                 <ros>
                     <argument>~/out:=scan</argument>

File: description/robot_core.xacro (robot description, xacro)
@@ -71,6 +71,4 @@
     <gazebo reference='left_front_wheel'>
         <material>Gazebo/Blue</material>
-        <mu1 value="0.001"/>
-        <mu2 value="0.001"/>
     </gazebo>
     <!-- RIGHT FRONT -->
@@ -99,6 +97,4 @@
     <gazebo reference='right_front_wheel'>
         <material>Gazebo/Blue</material>
-        <mu1 value="0.001"/>
-        <mu2 value="0.001"/>
     </gazebo>
     <!-- RIGHT REAR -->
@@ -106,5 +102,5 @@
         <parent link='base_link'/>
         <child link='right_rear_wheel'/>
-        <origin xyz = '0.5 0.35 -0.25' rpy='${pi/2} 0 0'/>
+        <origin xyz = '0.5 0.35 -0.25' rpy='-${pi/2} 0 0'/>
         <axis xyz='0 0 1'/>
     </joint>
@@ -132,5 +128,5 @@
         <parent link='base_link'/>
         <child link='left_rear_wheel'/>
-        <origin xyz = '0.5 -0.35 -0.25' rpy='-${pi/2} 0 0'/>
+        <origin xyz = '0.5 -0.35 -0.25' rpy='${pi/2} 0 0'/>
         <axis xyz='0 0 -1'/>
     </joint>

Commit message: 13/12 hard

File: description/gazebo_control.xacro (robot description, xacro)
@@ -4,6 +4,6 @@
         <plugin name="gz::sim::systems::DiffDrive" filename="gz-sim-diff-drive-system">
             <!-- Wheel Information -->
-            <left_joint>left_front_wheel_joint left_rear_wheel_joint</left_joint>
-            <right_joint>right_front_wheel_joint right_rear_wheel_joint</right_joint>
+            <left_joint>left_rear_wheel_joint</left_joint>
+            <right_joint>right_rear_wheel_joint</right_joint>
             <wheel_separation>0.297</wheel_separation>
             <wheel_radius>0.033</wheel_radius>
@@ -22,6 +22,6 @@
         name='gz::sim::systems::JointStatePublisher'>
             <topic>joint_states</topic>
-            <joint_name>left_front_wheel_joint left_rear_wheel_joint</joint_name>
-            <joint_name>right_front_wheel_joint right_rear_wheel_joint</joint_name>
+            <joint_name>left_rear_wheel_joint</joint_name>
+            <joint_name>right_rear_wheel_joint</joint_name>
         </plugin>
     </gazebo>

File: description/robot_core.xacro (robot description, xacro)
@@ -22,9 +22,9 @@
         <parent link='base_link'/>
         <child link='chassis'/>
-        <origin xyz='0 0 0'/>
+        <origin xyz='-0.226 0 0.25'/>
     </joint>
     <link name='chassis'>
         <visual>
-            <origin xyz= '0 0 0'/>
+            <origin xyz= '0.5 0 0.25'/>
             <geometry>
                 <box size= '1 0.7 0.5'/>
@@ -33,5 +33,5 @@
         </visual>
         <collision>
-            <origin xyz= '0 0 0'/>
+            <origin xyz= '0.5 0 0.25'/>
             <geometry>
                 <box size= '1 0.7 0.5'/>
@@ -39,5 +39,5 @@
         </collision>
         <xacro:inertial_box mass='1.4' x='1' y='0.7' z='0.5'>
-            <origin xyz= '0 0 0' rpy='0 0 0'/>
+            <origin xyz= '0.5 0 0.25' rpy='0 0 0'/>
         </xacro:inertial_box>
     </link>
@@ -50,6 +50,6 @@
         <parent link='base_link'/>
         <child link='left_front_wheel'/>
-        <origin xyz = '-0.5 -0.35 -0.25' rpy='-${pi/2} 0 0'/>
-        <axis xyz='0 0 -1'/>
+        <origin xyz = '0 0.1485 0' rpy='-${pi/2} 0 0'/>
+        <axis xyz='0 0 1'/>
     </joint>
     <link name='left_front_wheel'>
@@ -62,8 +62,8 @@
         <collision>
             <geometry>
-                <cylinder radius='0.15' length='0.04'/>
+                <sphere radius='0.15'/>
             </geometry>
         </collision>
-        <xacro:inertial_cylinder mass='0.01' length='0.04' radius='0.15'>
+        <xacro:inertial_cylinder mass='0.05' length='0.04' radius='0.15'>
             <origin xyz= '0 0 0' rpy='0 0 0'/>
         </xacro:inertial_cylinder>
@@ -71,4 +71,6 @@
     <gazebo reference='left_front_wheel'>
         <material>Gazebo/Blue</material>
+        <mu1 value="0.001"/>
+        <mu2 value="0.001"/>
     </gazebo>
     <!-- RIGHT FRONT -->
@@ -76,6 +78,6 @@
         <parent link='base_link'/>
         <child link='right_front_wheel'/>
-        <origin xyz = '-0.5 0.35 -0.25' rpy='${pi/2} 0 0'/>
-        <axis xyz='0 0 1'/>
+        <origin xyz = '0 -0.1485 0' rpy='${pi/2} 0 0'/>
+        <axis xyz='0 0 -1'/>
     </joint>
     <link name='right_front_wheel'>
@@ -88,8 +90,8 @@
         <collision>
             <geometry>
-                <cylinder radius='0.15' length='0.04'/>
+                <sphere radius='0.15'/>
             </geometry>
         </collision>
-        <xacro:inertial_cylinder mass='0.01' length='0.04' radius='0.15'>
+        <xacro:inertial_cylinder mass='0.05' length='0.04' radius='0.15'>
             <origin xyz= '0 0 0' rpy='0 0 0'/>
         </xacro:inertial_cylinder>
@@ -97,4 +99,6 @@
     <gazebo reference='right_front_wheel'>
         <material>Gazebo/Blue</material>
+        <mu1 value="0.001"/>
+        <mu2 value="0.001"/>
     </gazebo>
     <!-- RIGHT REAR -->
@@ -102,9 +106,9 @@
         <parent link='base_link'/>
         <child link='right_rear_wheel'/>
-        <origin xyz = '0.5 0.35 -0.25' rpy='-${pi/2} 0 0'/>
-        <axis xyz='0 0 1'/>
+        <origin xyz = '0 -0.1485 0' rpy='-${pi/2} 0 0'/>
+        <axis xyz='0 0 -1'/>
     </joint>
     <link name='right_rear_wheel'>
-        <visual>
+       <visual>
             <geometry>
                 <cylinder radius='0.15' length='0.04'/>
@@ -114,8 +118,8 @@
         <collision>
             <geometry>
-                <cylinder radius='0.15' length='0.04'/>
+                <sphere radius='0.15'/>
             </geometry>
         </collision>
-        <xacro:inertial_cylinder mass='0.01' length='0.04' radius='0.15'>
+        <xacro:inertial_cylinder mass='0.05' length='0.04' radius='0.15'>
             <origin xyz= '0 0 0' rpy='0 0 0'/>
         </xacro:inertial_cylinder>
@@ -128,9 +132,9 @@
         <parent link='base_link'/>
         <child link='left_rear_wheel'/>
-        <origin xyz = '0.5 -0.35 -0.25' rpy='${pi/2} 0 0'/>
-        <axis xyz='0 0 -1'/>
+        <origin xyz = '0 -0.1485 0' rpy='${pi/2} 0 0'/>
+        <axis xyz='0 0 1'/>
     </joint>
     <link name='left_rear_wheel'>
-        <visual>
+       <visual>
             <geometry>
                 <cylinder radius='0.15' length='0.04'/>
@@ -140,8 +144,8 @@
         <collision>
             <geometry>
-                <cylinder radius='0.15' length='0.04'/>
+                <sphere radius='0.15'/>
             </geometry>
         </collision>
-        <xacro:inertial_cylinder mass='0.01' length='0.04' radius='0.15'>
+        <xacro:inertial_cylinder mass='0.05' length='0.04' radius='0.15'>
             <origin xyz= '0 0 0' rpy='0 0 0'/>
         </xacro:inertial_cylinder>

Commit message: 14/01

File: description/gazebo_control.xacro (robot description, xacro)
@@ -4,20 +4,22 @@
         <plugin name="gz::sim::systems::DiffDrive" filename="gz-sim-diff-drive-system">
             <!-- Wheel Information -->
-            <left_joint>left_rear_wheel_joint</left_joint>
-            <right_joint>right_rear_wheel_joint</right_joint>
+            <left_joint>left_rear_wheel</left_joint>
+            <right_joint>right_rear_wheel</right_joint>
+            <left_joint>left_front_wheel</left_joint>
+            <right_joint>right_front_wheel</right_joint>
             <wheel_separation>0.297</wheel_separation>
             <wheel_radius>0.033</wheel_radius>
-            <!-- Limits -->
-            <max_wheel_acceleration>0.33</max_wheel_acceleration>
             <!-- Input -->
-            <topic>cmd_vel</topic>
+            <command_topic>cmd_vel</command_topic>
             <!-- Output -->
             <frame_id>odom</frame_id>
-            <child_frame_id>base_link</child_frame_id>
+            <robot_base_frame>base_link</robot_base_frame>
             <odom_topic>odom</odom_topic>
+            <publish_tf>true</publish_tf>
             <odom_publisher_frequency>30</odom_publisher_frequency>
             <tf_topic>/tf</tf_topic>
+            <use_velocity_feedback>true</use_velocity_feedback>
         </plugin>
-        <plugin filename='gz-sim-joint-state-publihser-system'
+        <plugin filename='gz-sim-joint-state-publisher-system'
         name='gz::sim::systems::JointStatePublisher'>
             <topic>joint_states</topic>

File: description/robot_core.xacro (robot description, xacro)
@@ -2,4 +2,5 @@
 <robot xmlns:xacro="http://www.ros.org/wiki/xacro" >
     <xacro:include filename='inertial_macros.xacro'/>
+    <xacro:property name="pi" value="3.141592653589793"/>
     <!-- Materials determine-->
     <material name='white'>
@@ -22,22 +23,22 @@
         <parent link='base_link'/>
         <child link='chassis'/>
-        <origin xyz='-0.226 0 0.25'/>
+        <origin xyz='0 0 0'/>
     </joint>
     <link name='chassis'>
         <visual>
-            <origin xyz= '0.5 0 0.25'/>
+            <origin xyz= '0 0 0.05' rpy='0 0 0'/>
             <geometry>
-                <box size= '1 0.7 0.5'/>
+                <box size= '0.23 0.16 0.05'/>
             </geometry>
             <material name='white'/>
         </visual>
         <collision>
-            <origin xyz= '0.5 0 0.25'/>
+            <origin xyz= '0 0 0.05' rpy='0 0 0'/>
             <geometry>
-                <box size= '1 0.7 0.5'/>
+                <box size= '0.23 0.16 0.05'/>
             </geometry>
         </collision>
-        <xacro:inertial_box mass='1.4' x='1' y='0.7' z='0.5'>
-            <origin xyz= '0.5 0 0.25' rpy='0 0 0'/>
+        <xacro:inertial_box mass='1.4' x='0.23' y='0.16' z='0.05'>
+            <origin xyz= '0 0 0.05' rpy='0 0 0'/>
         </xacro:inertial_box>
     </link>
@@ -46,37 +47,9 @@
     </gazebo>
     <!-- Wheels -->
-    <!-- LEFT FRONT -->
-    <joint name="left_front_wheel_joint" type='continuous'>
-        <parent link='base_link'/>
-        <child link='left_front_wheel'/>
-        <origin xyz = '0 0.1485 0' rpy='-${pi/2} 0 0'/>
-        <axis xyz='0 0 1'/>
-    </joint>
-    <link name='left_front_wheel'>
-        <visual>
-            <geometry>
-                <cylinder radius='0.15' length='0.04'/>
-            </geometry>
-            <material name='blue'/>
-        </visual>
-        <collision>
-            <geometry>
-                <sphere radius='0.15'/>
-            </geometry>
-        </collision>
-        <xacro:inertial_cylinder mass='0.05' length='0.04' radius='0.15'>
-            <origin xyz= '0 0 0' rpy='0 0 0'/>
-        </xacro:inertial_cylinder>
-    </link>
-    <gazebo reference='left_front_wheel'>
-        <material>Gazebo/Blue</material>
-        <mu1 value="0.001"/>
-        <mu2 value="0.001"/>
-    </gazebo>
-    <!-- RIGHT FRONT -->
+    <!-- ##########################################      RIGHT FRONT       ##########################################-->
     <joint name="right_front_wheel_joint" type='continuous'>
-        <parent link='base_link'/>
+        <parent link='chassis'/>
         <child link='right_front_wheel'/>
-        <origin xyz = '0 -0.1485 0' rpy='${pi/2} 0 0'/>
+        <origin xyz='0.1425 -0.1425 0' rpy='-${pi/2} 0 0'/>
         <axis xyz='0 0 -1'/>
     </joint>
@@ -99,12 +72,10 @@
     <gazebo reference='right_front_wheel'>
         <material>Gazebo/Blue</material>
-        <mu1 value="0.001"/>
-        <mu2 value="0.001"/>
     </gazebo>
-    <!-- RIGHT REAR -->
+     <!-- ##########################################      RIGHT REAR       ########################################## -->
     <joint name="right_rear_wheel_joint" type='continuous'>
-        <parent link='base_link'/>
+        <parent link='chassis'/>
         <child link='right_rear_wheel'/>
-        <origin xyz = '0 -0.1485 0' rpy='-${pi/2} 0 0'/>
+        <origin xyz = '-0.1425 -0.1425 0' rpy='-${pi/2} 0 0'/>
         <axis xyz='0 0 -1'/>
     </joint>
@@ -128,9 +99,35 @@
         <material>Gazebo/Blue</material>
     </gazebo>
-    <!-- LEFT REAR -->
+    <!-- ##########################################      LEFT FRONT       ########################################## -->
+    <joint name="left_front_wheel_joint" type='continuous'>
+        <parent link='chassis'/>
+        <child link='left_front_wheel'/>
+        <origin xyz='0.1425 0.1425 0' rpy='${pi/2} 0 0'/>
+        <axis xyz='0 0 1'/>
+    </joint>
+    <link name='left_front_wheel'>
+        <visual>
+            <geometry>
+                <cylinder radius='0.15' length='0.04'/>
+            </geometry>
+            <material name='blue'/>
+        </visual>
+        <collision>
+            <geometry>
+                <sphere radius='0.15'/>
+            </geometry>
+        </collision>
+        <xacro:inertial_cylinder mass='0.05' length='0.04' radius='0.15'>
+            <origin xyz= '0 0 0' rpy='0 0 0'/>
+        </xacro:inertial_cylinder>
+    </link>
+    <gazebo reference='left_front_wheel'>
+        <material>Gazebo/Blue</material>
+    </gazebo>
+    <!-- ##########################################      LEFT REAR       ########################################## -->
     <joint name="left_rear_wheel_joint" type='continuous'>
         <parent link='base_link'/>
         <child link='left_rear_wheel'/>
-        <origin xyz = '0 -0.1485 0' rpy='${pi/2} 0 0'/>
+        <origin xyz = '-0.1425 0.1425 0' rpy='${pi/2} 0 0'/>
         <axis xyz='0 0 1'/>
     </joint>
